File: pcb/Laser_Shield_Eth.brd (EAGLE design)
At the start: 68.6 x 53.3 mm, 61 parts, among them IC1 CAT811TTBI-CT3, IC11 74LVC1G14DBV, IC2 MC33269ST-3, IC3 MC33269D-3, IC4 W5100, J4 JUMPER_SOLDER_1X2, Q1 25MHz, U1 SN74LVC2G241DCUT, X1 22-23-2031, X2 22-23-2031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

Commit message: pcb done?
Parts:
- removed FULLD: (no value), led:CHIPLED_0805
- added J5, J6: JUMPER_SOLDER_1X2, parts:JUMPER_SOLDER_1X2
- added Q2: MOSFET-NCHANNELSMD, SparkFun-DiscreteSemi:SOT23-3
- added R13: 100k, SmartPrj:R0603-ROUND
- moved C3 2.42 mm to (54.0, 33.1), turned to 90 degrees
- moved C16 1.35 mm to (51.3, 10.4), turned to 0 degrees
- moved R1 0.76 mm to (53.1, 29.7)
- renumbered X1 to SERVO, X2 to LASER, X3 to CAM
Connections:
- new net N$13: J6.2, Q2.1, R13.2
- new net N$14: J5.2, LASER.1, Q2.3
- new net N$15: J1.6, RN1.1
- net GND: now also J5.1, Q2.2, R13.1; no longer LASER.1
- net LASER_CTRL: now also J6.1
- net SCK: no longer RN1.1
Routing:
- net SCK: track 83.0 -> 43.1 mm, vias 4 -> 1
- net N$13: track 0.00 -> 17.0 mm, vias 0 -> 2
- net N$15: track 0.00 -> 13.1 mm
- net N$14: track 0.00 -> 12.3 mm
- net RESET: track 110.4 -> 104.1 mm, vias 6 -> 5
- net LASER_CTRL: track 48.3 -> 50.9 mm
- net +3V3A: track 49.9 -> 47.5 mm
- net +5V: track 124.1 -> 122.2 mm
- net N$1: track 3.22 -> 4.17 mm
- net GND: track 137.2 -> 137.6 mm, vias 38 -> 39
Other:
- board text added: "* * * * 9 8"
- board text added: "0 1 2 3 * *"
- board text added: "12V"
- board text added: "5V"
- board text added: "7 6 * * * * * *"
- board text added: "RST"
- board text removed: "(*=PWM)"
- board text removed: "*"
- board text removed: "0 1 2 3 4 5"
- board text removed: "1 1 1 1"
- board text removed: "3 2 1 0 9 8"
- board text removed: "5V Gnd 12V"
- board text removed: "7 6 5 4 3 2 1 0"
- board text removed: "ANALOG IN"
- board text removed: "Arduino"
- board text removed: "D.Cuartielles"
- board text removed: "D.Mellis"
- board text removed: "G.Martino"
- board text removed: "M.Banzi"
- board text removed: "RES"
- board text removed: "RX"
- board text removed: "T.Igoe"
- board text removed: "TM"
- board text removed: "TX"
- board text removed: "www.arduino.cc"
